File: rp2040_custom_devboard.kicad_pcb (KiCad board)
At the start: 2 copper layers, 34 parts, among them J1 USB_B_Micro, J2 Conn_02x18_Odd_Even, J3 Conn_02x18_Odd_Even, J4 Conn_01x02, U1 NCP1117-3.3_SOT223, U2 W25Q128JVS, U3 RP2040, Y1 ABM8-272-T3

Commit message: REV1
Parts:
- added G***: LOGO, LOGO, F.Cu at (153.6, 118.6)
- moved C14 59.5 mm to (155.1, 106.9)
- moved C13 51.3 mm to (155.1, 104.4)
- moved C6 51.0 mm to (139.9, 91.8), turned to 90 degrees
- moved H1 50.6 mm to (127.0, 84.5)
- moved C3 49.7 mm to (151.8, 104.8)
- moved C1 46.5 mm to (155.8, 88.5)
- moved C2 46.4 mm to (157.2, 102.5), turned to -90 degrees
- moved C8 46.4 mm to (151.3, 94.8)
- moved U1 46.3 mm to (157.2, 95.5)
- moved H3 45.1 mm to (127.0, 126.5)
- moved C9 44.5 mm to (151.3, 97.3), turned to 180 degrees
- moved R4 44.0 mm to (138.0, 94.5)
- moved C4 42.2 mm to (149.3, 104.8)
- moved R3 41.9 mm to (134.0, 94.5)
- moved J1 41.5 mm to (143.0, 84.5)
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Connections:
- C2 pad 1: +3V3 -> unconnected-(C2-Pad1)
- C2 pad 2: GND -> unconnected-(C2-Pad2)
Routing:
- net GND: track 0.00 -> 72.5 mm, vias 0 -> 6
- net /GPIO29_ADC3: track 0.00 -> 39.3 mm
- net /GPIO0: track 0.00 -> 37.9 mm
- net /GPIO28_ADC2: track 0.00 -> 37.7 mm
- net /GPIO27_ADC1: track 0.00 -> 36.4 mm
- net /GPIO1: track 0.00 -> 35.7 mm
- net /GPIO26_ADC0: track 0.00 -> 34.3 mm
- net /GPIO2: track 0.00 -> 33.6 mm
- net /GPIO25: track 0.00 -> 32.1 mm
- net /QSPI_SS: track 0.00 -> 31.5 mm
- net /GPIO3: track 0.00 -> 31.5 mm
- net /GPIO24: track 0.00 -> 30.0 mm
- net /GPIO4: track 0.00 -> 29.3 mm
- net /GPIO23: track 0.00 -> 27.8 mm
- net /GPIO5: track 0.00 -> 27.2 mm
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- added copper zone on F.Cu, net +1V1
- added copper zone on F.Cu, net +3V3
- added copper zone on B.Cu, net GND
- added copper zone on F.Cu, net VBUS
Other:
- board outline added: 58 x 49.9 mm
- copper layers 2 -> 4
- board text added: "3V3"
- board text added: "GND"
- board text added: "GP0"
- board text added: "GP1"
- board text added: "GP10"
- board text added: "GP11"
- board text added: "GP12"
- board text added: "GP13"
- board text added: "GP14"
- board text added: "GP15"
- board text added: "GP16"
- board text added: "GP17"
- board text added: "GP18"
- board text added: "GP19"
- board text added: "GP2"
- board text added: "GP20"
- board text added: "GP21"
- board text added: "GP22"
- board text added: "GP23"
- board text added: "GP24"
- board text added: "GP25"
- board text added: "GP26"
- board text added: "GP27"
- board text added: "GP28"
- board text added: "GP29"
- board text added: "GP3"
- board text added: "GP4"
- board text added: "GP5"
- board text added: "GP6"
- board text added: "GP7"
- board text added: "GP8"
- board text added: "GP9"
- board text added: "Guster32 RP2040 Test Build REV1 2025-06-22"
- board text added: "JLCJLCJLCJLC"
- board text added: "Outer Row GND"
- board text added: "RUN"
- board text added: "SWCLK"
- board text added: "SWD"
